File: minimal_max17570/minimal_max17570.kicad_sch (KiCad schematic)
At the start: 0 parts

Commit message: backup
Parts:
- added C1: 1 µF, capacitor_footprints:C_0402_1005Metric, symbol CAPACITORS_C1005X6S1C_DATA_BASE:C_C1005X6S1C105K050BC
- added C2: 10 µF, capacitor_footprints:C_1206_3216Metric, symbol CAPACITORS_CL31B_DATA_BASE:C_CL31B106KBHNNN#
- added C3: 1 µF, capacitor_footprints:C_0805_2012Metric, symbol CAPACITORS_GRJ21BC72A_DATA_BASE:C_GRJ21BC72A105KE11L
- added L1: 100.0 µH, inductor_footprints:74404054, symbol INDUCTORS_74404054_DATA_BASE:L_74404054101
- added R1: 40.2 kΩ, resistor_footprints:R_0402_1005Metric, symbol RESISTORS_ERJ-2RKF_DATA_BASE:R_ERJ-2RKF4022X
- added R2: 9.76 kΩ, resistor_footprints:R_0402_1005Metric, symbol RESISTORS_ERJ-2RKF_DATA_BASE:R_ERJ-2RKF9761X
- added R3: 499 kΩ, resistor_footprints:R_0402_1005Metric, symbol RESISTORS_ERJ-2RKF_DATA_BASE:R_ERJ-2RKF4993X
- added R4: 1 kΩ, resistor_footprints:R_0402_1005Metric, symbol UNITED_RESISTORS_DATA_BASE:R_ERJ-2RKF1001X
- added R5: 3.32 MΩ, resistor_footprints:R_0402_1005Metric, symbol RESISTORS_RC0402FR-07_DATA_BASE:R_RC0402FR-073M32L
- added R6: 294 kΩ, resistor_footprints:R_0402_1005Metric, symbol RESISTORS_ERJ-2RKF_DATA_BASE:R_ERJ-2RKF2943X
- added U1: MAX17570FATA+, analog_devices_footprints:21-100514_T822C&plus_6C_ADI, symbol UNITED_IC_ADI:U_MAX17570FATA+
Connections:
- new net: R2.1, U1.5 (RT/SYNC)
- new net EN: R5.2, R6.1, U1.2 (EN/UVLO)
- new net FB: R1.1, R3.2, U1.4 (VOUT/FB)
- new net GND: C1.2, C2.2, C3.2, R1.2, R2.2, R6.2, U1.7 (GND)
- new net LX: L1.1, U1.8 (LX)
- new net VCC: C1.1, R4.1, U1.3 (VCC)
- new net VIN: C3.1, R5.1, U1.1 (VIN)
- new net VOUT: C2.1, L1.2, R3.1
- new net ~{RESET}: R4.2, U1.6 (~{RESET})

Commit message: backup
Parts:
- R4: symbol UNITED_RESISTORS_DATA_BASE:R_ERJ-2RKF1001X -> RESISTORS_ERJ-2RKF_DATA_BASE:R_ERJ-2RKF1001X
Changed lines of the file:
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@@
 		(dnp no)
 		(fields_autoplaced yes)
-		(property "Reference" "#PWR02"
+		(property "Reference" "#PWR2"
 			(at 203.2 97.79 0)
 			(effects
@@
 			(project "minimal_max17570"
 				(path "/92f3cd93-efd9-4305-a902-cde57c556096"
-					(reference "#PWR02")
+					(reference "#PWR2")
 					(unit 1)
 				)
@@
 		(dnp no)
 		(fields_autoplaced yes)
-		(property "Reference" "#PWR04"
+		(property "Reference" "#PWR4"
 			(at 190.5 118.11 0)
 			(effects
@@
 			(project "minimal_max17570"
 				(path "/92f3cd93-efd9-4305-a902-cde57c556096"
-					(reference "#PWR04")
+					(reference "#PWR4")
 					(unit 1)
 				)
@@
 		(dnp no)
 		(fields_autoplaced yes)
-		(property "Reference" "#PWR06"
+		(property "Reference" "#PWR6"
 			(at 111.76 97.79 0)
 			(effects
@@
 			(project "minimal_max17570"
 				(path "/92f3cd93-efd9-4305-a902-cde57c556096"
-					(reference "#PWR06")
+					(reference "#PWR6")
 					(unit 1)
 				)
@@
 	)
 	(symbol
-		(lib_id "UNITED_RESISTORS_DATA_BASE:R_ERJ-2RKF1001X")
+		(lib_id "RESISTORS_ERJ-2RKF_DATA_BASE:R_ERJ-2RKF1001X")
 		(at 170.18 110.49 90)
 		(mirror x)
@@
 		(dnp no)
 		(fields_autoplaced yes)
-		(property "Reference" "#PWR03"
+		(property "Reference" "#PWR3"
 			(at 134.62 135.89 0)
 			(effects
@@
 			(project "minimal_max17570"
 				(path "/92f3cd93-efd9-4305-a902-cde57c556096"
-					(reference "#PWR03")
+					(reference "#PWR3")
 					(unit 1)
 				)
@@
 		(dnp no)
 		(fields_autoplaced yes)
-		(property "Reference" "#PWR07"
+		(property "Reference" "#PWR7"
 			(at 127 118.11 0)
 			(effects
@@
 			(project "minimal_max17570"
 				(path "/92f3cd93-efd9-4305-a902-cde57c556096"
-					(reference "#PWR07")
+					(reference "#PWR7")
 					(unit 1)
 				)
@@
 		(dnp no)
 		(fields_autoplaced yes)
-		(property "Reference" "#PWR01"
+		(property "Reference" "#PWR1"
 			(at 152.4 129.54 0)
 			(effects
@@
 			(project ""
 				(path "/92f3cd93-efd9-4305-a902-cde57c556096"
-					(reference "#PWR01")
+					(reference "#PWR1")
 					(unit 1)
 				)
@@
 		(dnp no)
 		(fields_autoplaced yes)
-		(property "Reference" "#PWR05"
+		(property "Reference" "#PWR5"
 			(at 162.56 78.74 0)
 			(effects
@@
 			(project "minimal_max17570"
 				(path "/92f3cd93-efd9-4305-a902-cde57c556096"
-					(reference "#PWR05")
+					(reference "#PWR5")
 					(unit 1)
 				)

Commit message: backup
Parts:
- added C2, C4: 100 nF, capacitor_footprints:C_0603_1608Metric, symbol CAPACITORS_C1608X7S2A_DATA_BASE:C_C1608X7S2A104K080AB
- added C3: 220 pF, capacitor_footprints:C_0402_1005Metric, symbol CAPACITORS_CGA2B2NP02A_DATA_BASE:C_CGA2B2NP02A221J050BA
- added TP1, TP2, TP3, TP4, TP5: TestPoint, test_point_footprints:TestPoint_THTPad_Castelated, symbol UNITED_TEST_POINTS:TestPoint_Castelated
- renumbered C3 to C1, C1 to C5, C2 to C6, R6 to R1, R5 to R2, R1 to R3, R3 to R4, R2 to R5, R4 to R6
Connections:
- net GND: now also C2.2, C3.2, C4.2, TP2.1, TP4.1
- net VIN: now also C2.1, C3.1, TP1.1
- net VOUT: now also C4.1, TP5.1
- net ~{RESET}: now also TP3.1
Other:
- moved on the sheet: C1, C5, C6, L1, R1, R2, R3, R4, R5, R6, U1

Commit message: backup
Parts:
- renumbered C1 to C100, C2 to C101, C3 to C102, C4 to C103, C5 to C104, C6 to C105, L1 to L100, R1 to R100, R2 to R101, R3 to R102, R4 to R103, R5 to R104, R6 to R105, TP1 to TP100, TP2 to TP101, TP3 to TP102, TP4 to TP103, TP5 to TP104, U1 to U100
Connections:
- net VIN renamed MAX17570_VIN
- net VOUT renamed MAX17570_VOUT
- net ~{RESET} renamed ~{MAX17570_RESET}
Changed lines of the file:
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@@
 		)
 	)
-	(label "~{RESET}"
+	(label "~{MAX17570_RESET}"
 		(at 172.72 86.36 0)
 		(effects
@@
 		)
 	)
-	(label "VIN"
-		(at 130.81 86.36 180)
+	(label "MAX17570_VIN"
+		(at 137.16 86.36 180)
 		(effects
 			(font
@@
 		)
 	)
-	(label "VOUT"
+	(label "MAX17570_VOUT"
 		(at 193.04 99.06 0)
 		(effects
@@
 		(on_board yes)
 		(dnp no)
-		(property "Reference" "C1"
+		(property "Reference" "C100"
 			(at 72.39 90.1699 90)
 			(effects
@@
 			(project ""
 				(path "/92f3cd93-efd9-4305-a902-cde57c556096"
-					(reference "C1")
+					(reference "C100")
 					(unit 1)
 				)
@@
 		(on_board yes)
 		(dnp no)
-		(property "Reference" "R5"
+		(property "Reference" "R104"
 			(at 134.62 109.2199 90)
 			(effects
@@
 			(project ""
 				(path "/92f3cd93-efd9-4305-a902-cde57c556096"
-					(reference "R5")
+					(reference "R104")
 					(unit 1)
 				)
@@
 		(dnp no)
 		(fields_autoplaced yes)
-		(property "Reference" "R6"
+		(property "Reference" "R105"
 			(at 170.18 78.7399 90)
 			(effects
@@
 			(project "minimal_max17570"
 				(path "/92f3cd93-efd9-4305-a902-cde57c556096"
-					(reference "R6")
+					(reference "R105")
 					(unit 1)
 				)
@@
 		(dnp no)
 		(fields_autoplaced yes)
-		(property "Reference" "C5"
+		(property "Reference" "C104"
 			(at 147.32 68.58 0)
 			(effects
@@
 			(project ""
 				(path "/92f3cd93-efd9-4305-a902-cde57c556096"
-					(reference "C5")
+					(reference "C104")
 					(unit 1)
 				)
@@
 		(dnp no)
 		(fields_autoplaced yes)
-		(property "Reference" "L1"
+		(property "Reference" "L100"
 			(at 177.8 92.71 0)
 			(effects
@@
 			(project ""
 				(path "/92f3cd93-efd9-4305-a902-cde57c556096"
-					(reference "L1")
+					(reference "L100")
 					(unit 1)
 				)
@@
 		(dnp no)
 		(fields_autoplaced yes)
-		(property "Reference" "R4"
+		(property "Reference" "R103"
 			(at 190.5 104.1399 90)
 			(effects
@@
 			(project ""
 				(path "/92f3cd93-efd9-4305-a902-cde57c556096"
-					(reference "R4")
+					(reference "R103")
 					(unit 1)
 				)
@@
 		(dnp no)
 		(fields_autoplaced yes)
-		(property "Reference" "TP5"
+		(property "Reference" "TP104"
 			(at 231.902 96.52 90)
 			(effects
@@
 			(project "minimal_max17570"
 				(path "/92f3cd93-efd9-4305-a902-cde57c556096"
-					(reference "TP5")
+					(reference "TP104")
 					(unit 1)
 				)
@@
 		(on_board yes)
 		(dnp no)
-		(property "Reference" "R2"
+		(property "Reference" "R101"
 			(at 119.38 91.4399 90)
 			(effects
@@
 			(project ""
 				(path "/92f3cd93-efd9-4305-a902-cde57c556096"
-					(reference "R2")
+					(reference "R101")
 					(unit 1)
 				)
@@
 		(dnp no)
 		(fields_autoplaced yes)
-		(property "Reference" "C6"
+		(property "Reference" "C105"
 			(at 222.25 102.8699 90)
 			(effects
@@
 			(project ""
 				(path "/92f3cd93-efd9-4305-a902-cde57c556096"
-					(reference "C6")
+					(reference "C105")
 					(unit 1)
 				)
@@
 		(dnp no)
 		(fields_autoplaced yes)
-		(property "Reference" "C4"
+		(property "Reference" "C103"
 			(at 207.01 102.8699 90)
 			(effects
@@
 			(project ""
 				(path "/92f3cd93-efd9-4305-a902-cde57c556096"
-					(reference "C4")
+					(reference "C103")
 					(unit 1)
 				)
@@
 		(on_board yes)
 		(dnp no)
-		(property "Reference" "C3"
+		(property "Reference" "C102"
 			(at 102.87 90.1699 90)
 			(effects
@@
 			(project ""
 				(path "/92f3cd93-efd9-4305-a902-cde57c556096"
-					(reference "C3")
+					(reference "C102")
 					(unit 1)
 				)
@@
 		(dnp no)
 		(fields_autoplaced yes)
-		(property "Reference" "U1"
+		(property "Reference" "U100"
 			(at 154.5433 121.92 0)
 			(effects
@@
 			(project ""
 				(path "/92f3cd93-efd9-4305-a902-cde57c556096"
-					(reference "U1")
+					(reference "U100")
 					(unit 1)
 				)
@@
 		(on_board yes)
 		(dnp no)
-		(property "Reference" "C2"
+		(property "Reference" "C101"
 			(at 87.63 90.1699 90)
 			(effects
@@
 			(project "minimal_max17570"
 				(path "/92f3cd93-efd9-4305-a902-cde57c556096"
-					(reference "C2")
+					(reference "C101")
 					(unit 1)
 				)
@@
 		(dnp no)
 		(fields_autoplaced yes)
-		(property "Reference" "TP3"
+		(property "Reference" "TP102"
 			(at 231.902 83.82 90)
 			(effects
@@
 			(project "minimal_max17570"
 				(path "/92f3cd93-efd9-4305-a902-cde57c556096"
-					(reference "TP3")
+					(reference "TP102")
 					(unit 1)
 				)
@@
 		(dnp no)
 		(fields_autoplaced yes)
-		(property "Reference" "TP2"
+		(property "Reference" "TP101"
 			(at 62.738 91.44 90)
 			(effects
@@
 			(project "minimal_max17570"
 				(path "/92f3cd93-efd9-4305-a902-cde57c556096"
-					(reference "TP2")
+					(reference "TP101")
 					(unit 1)
 				)
@@
 		(dnp no)
 		(fields_autoplaced yes)
-		(property "Reference" "TP1"
+		(property "Reference" "TP100"
 			(at 62.738 83.82 90)
 			(effects
@@
 			(project ""
 				(path "/92f3cd93-efd9-4305-a902-cde57c556096"
-					(reference "TP1")
+					(reference "TP100")
 					(unit 1)
 				)
@@
 		(dnp no)
 		(fields_autoplaced yes)
-		(property "Reference" "TP4"
+		(property "Reference" "TP103"
 			(at 231.902 104.14 90)
 			(effects
@@
 			(project "minimal_max17570"
 				(path "/92f3cd93-efd9-4305-a902-cde57c556096"
-					(reference "TP4")
+					(reference "TP103")
 					(unit 1)
 				)
@@
 		(on_board yes)
 		(dnp no)
-		(property "Reference" "R1"
+		(property "Reference" "R100"
 			(at 119.38 104.1399 90)
 			(effects
@@
 			(project ""
 				(path "/92f3cd93-efd9-4305-a902-cde57c556096"
-					(reference "R1")
+					(reference "R100")
 					(unit 1)
 				)
@@
 		(dnp no)
 		(fields_autoplaced yes)
-		(property "Reference" "R3"
+		(property "Reference" "R102"
 			(at 190.5 119.3799 90)
 			(effects
@@
 			(project ""
 				(path "/92f3cd93-efd9-4305-a902-cde57c556096"
-					(reference "R3")
+					(reference "R102")
 					(unit 1)
 				)

Commit message: backup
Parts:
- renumbered C100 to C1, C101 to C2, C102 to C3, C103 to C4, C104 to C5, C105 to C6, L100 to L1, R100 to R1, R101 to R2, R102 to R3, R103 to R4, R104 to R5, R105 to R6, TP100 to TP1, TP101 to TP2, TP102 to TP3, TP103 to TP4, TP104 to TP5, U100 to U1
Changed lines of the file:
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@@
 		(on_board yes)
 		(dnp no)
-		(property "Reference" "C100"
+		(property "Reference" "C1"
 			(at 72.39 90.1699 90)
 			(effects
@@
 			(project ""
 				(path "/92f3cd93-efd9-4305-a902-cde57c556096"
-					(reference "C100")
+					(reference "C1")
 					(unit 1)
 				)
@@
 		(on_board yes)
 		(dnp no)
-		(property "Reference" "R104"
+		(property "Reference" "R5"
 			(at 134.62 109.2199 90)
 			(effects
@@
 			(project ""
 				(path "/92f3cd93-efd9-4305-a902-cde57c556096"
-					(reference "R104")
+					(reference "R5")
 					(unit 1)
 				)
@@
 		(dnp no)
 		(fields_autoplaced yes)
-		(property "Reference" "R105"
+		(property "Reference" "R6"
 			(at 170.18 78.7399 90)
 			(effects
@@
 			(project "minimal_max17570"
 				(path "/92f3cd93-efd9-4305-a902-cde57c556096"
-					(reference "R105")
+					(reference "R6")
 					(unit 1)
 				)
@@
 		(dnp no)
 		(fields_autoplaced yes)
-		(property "Reference" "C104"
+		(property "Reference" "C5"
 			(at 147.32 68.58 0)
 			(effects
@@
 			(project ""
 				(path "/92f3cd93-efd9-4305-a902-cde57c556096"
-					(reference "C104")
+					(reference "C5")
 					(unit 1)
 				)
@@
 		(dnp no)
 		(fields_autoplaced yes)
-		(property "Reference" "L100"
+		(property "Reference" "L1"
 			(at 177.8 92.71 0)
 			(effects
@@
 			(project ""
 				(path "/92f3cd93-efd9-4305-a902-cde57c556096"
-					(reference "L100")
+					(reference "L1")
 					(unit 1)
 				)
@@
 		(dnp no)
 		(fields_autoplaced yes)
-		(property "Reference" "R103"
+		(property "Reference" "R4"
 			(at 190.5 104.1399 90)
 			(effects
@@
 			(project ""
 				(path "/92f3cd93-efd9-4305-a902-cde57c556096"
-					(reference "R103")
+					(reference "R4")
 					(unit 1)
 				)
@@
 		(dnp no)
 		(fields_autoplaced yes)
-		(property "Reference" "TP104"
+		(property "Reference" "TP5"
 			(at 231.902 96.52 90)
 			(effects
@@
 			(project "minimal_max17570"
 				(path "/92f3cd93-efd9-4305-a902-cde57c556096"
-					(reference "TP104")
+					(reference "TP5")
 					(unit 1)
 				)
@@
 		(on_board yes)
 		(dnp no)
-		(property "Reference" "R101"
+		(property "Reference" "R2"
 			(at 119.38 91.4399 90)
 			(effects
@@
 			(project ""
 				(path "/92f3cd93-efd9-4305-a902-cde57c556096"
-					(reference "R101")
+					(reference "R2")
 					(unit 1)
 				)
@@
 		(dnp no)
 		(fields_autoplaced yes)
-		(property "Reference" "C105"
+		(property "Reference" "C6"
 			(at 222.25 102.8699 90)
 			(effects
@@
 			(project ""
 				(path "/92f3cd93-efd9-4305-a902-cde57c556096"
-					(reference "C105")
+					(reference "C6")
 					(unit 1)
 				)
@@
 		(dnp no)
 		(fields_autoplaced yes)
-		(property "Reference" "C103"
+		(property "Reference" "C4"
 			(at 207.01 102.8699 90)
 			(effects
@@
 			(project ""
 				(path "/92f3cd93-efd9-4305-a902-cde57c556096"
-					(reference "C103")
+					(reference "C4")
 					(unit 1)
 				)
@@
 		(on_board yes)
 		(dnp no)
-		(property "Reference" "C102"
+		(property "Reference" "C3"
 			(at 102.87 90.1699 90)
 			(effects
@@
 			(project ""
 				(path "/92f3cd93-efd9-4305-a902-cde57c556096"
-					(reference "C102")
+					(reference "C3")
 					(unit 1)
 				)
@@
 		(dnp no)
 		(fields_autoplaced yes)
-		(property "Reference" "U100"
+		(property "Reference" "U1"
 			(at 154.5433 121.92 0)
 			(effects
@@
 			(project ""
 				(path "/92f3cd93-efd9-4305-a902-cde57c556096"
-					(reference "U100")
+					(reference "U1")
 					(unit 1)
 				)
@@
 		(on_board yes)
 		(dnp no)
-		(property "Reference" "C101"
+		(property "Reference" "C2"
 			(at 87.63 90.1699 90)
 			(effects
@@
 			(project "minimal_max17570"
 				(path "/92f3cd93-efd9-4305-a902-cde57c556096"
-					(reference "C101")
+					(reference "C2")
 					(unit 1)
 				)
@@
 		(dnp no)
 		(fields_autoplaced yes)
-		(property "Reference" "TP102"
+		(property "Reference" "TP3"
 			(at 231.902 83.82 90)
 			(effects
@@
 			(project "minimal_max17570"
 				(path "/92f3cd93-efd9-4305-a902-cde57c556096"
-					(reference "TP102")
+					(reference "TP3")
 					(unit 1)
 				)
@@
 		(dnp no)
 		(fields_autoplaced yes)
-		(property "Reference" "TP101"
+		(property "Reference" "TP2"
 			(at 62.738 91.44 90)
 			(effects
@@
 			(project "minimal_max17570"
 				(path "/92f3cd93-efd9-4305-a902-cde57c556096"
-					(reference "TP101")
+					(reference "TP2")
 					(unit 1)
 				)
@@
 		(dnp no)
 		(fields_autoplaced yes)
-		(property "Reference" "TP100"
+		(property "Reference" "TP1"
 			(at 62.738 83.82 90)
 			(effects
@@
 			(project ""
 				(path "/92f3cd93-efd9-4305-a902-cde57c556096"
-					(reference "TP100")
+					(reference "TP1")
 					(unit 1)
 				)
@@
 		(dnp no)
 		(fields_autoplaced yes)
-		(property "Reference" "TP103"
+		(property "Reference" "TP4"
 			(at 231.902 104.14 90)
 			(effects
@@
 			(project "minimal_max17570"
 				(path "/92f3cd93-efd9-4305-a902-cde57c556096"
-					(reference "TP103")
+					(reference "TP4")
 					(unit 1)
 				)
@@
 		(on_board yes)
 		(dnp no)
-		(property "Reference" "R100"
+		(property "Reference" "R1"
 			(at 119.38 104.1399 90)
 			(effects
@@
 			(project ""
 				(path "/92f3cd93-efd9-4305-a902-cde57c556096"
-					(reference "R100")
+					(reference "R1")
 					(unit 1)
 				)
@@
 		(dnp no)
 		(fields_autoplaced yes)
-		(property "Reference" "R102"
+		(property "Reference" "R3"
 			(at 190.5 119.3799 90)
 			(effects
@@
 			(project ""
 				(path "/92f3cd93-efd9-4305-a902-cde57c556096"
-					(reference "R102")
+					(reference "R3")
 					(unit 1)
 				)
